Commit message: human can generate trajectory, but looks abnormal

File: hierarchial_simulation/src/moveit_human_config/config/gazebo_XSensStyleModel_template.urdf (robot description, URDF)
Before this commit: robot XSensStyleModel_template, 51 links, 50 joints
Links:
- link LeftHand: geometry collision box size=0.06145 0.16718 0.039266; visual box size=0.06145 0.16718 0.039266

Commit message: add fanuc1

File: hierarchial_simulation/src/moveit_human_config/config/gazebo_XSensStyleModel_template.urdf (robot description, URDF)
Before this commit: robot XSensStyleModel_template, 51 links, 50 joints
Joints:
- joint jLeftWrist_rotx: limit lower=-1.0472 upper=0.872665 effort=30 velocity=1.0 -> (none)

File: hierarchial_simulation/src/moveit_human_config/config/humanSubject01_48dof.urdf (robot description, URDF)
Before this commit: robot XSensStyleModel_template, 52 links, 51 joints
Joints:
- joint jC1Head_rotx: limit lower=-0.610865 upper=0.610865 effort=100 velocity=1.0 -> lower=-0.610865 upper=0.610865 effort=100 velocity=2.0
- joint jC1Head_roty: limit lower=-0.436332 upper=0.174533 effort=100 velocity=1.0 -> lower=-0.436332 upper=0.174533 effort=100 velocity=2.0
- joint jL1T12_rotx: limit lower=-0.610865 upper=0.610865 effort=100 velocity=1.0 -> lower=-0.610865 upper=0.610865 effort=100 velocity=2.0
- joint jL1T12_roty: limit lower=-0.523599 upper=1.309 effort=100 velocity=1.0 -> lower=-0.523599 upper=1.309 effort=100 velocity=2.0
- joint jL4L3_rotx: limit lower=-0.610865 upper=0.610865 effort=8000 velocity=1.0 -> lower=-0.610865 upper=0.610865 effort=8000 velocity=2.0
- joint jL4L3_roty: limit lower=-0.523599 upper=1.309 effort=8000 velocity=1.0 -> lower=-0.523599 upper=1.309 effort=8000 velocity=2.0
- joint jL5S1_rotx: limit lower=-0.610865 upper=0.610865 effort=100 velocity=1.0 -> lower=-0.610865 upper=0.610865 effort=100 velocity=2.0
- joint jL5S1_roty: limit lower=-0.523599 upper=1.309 effort=60 velocity=1.0 -> lower=-0.523599 upper=1.309 effort=60 velocity=2.0
- joint jLeftAnkle_rotx: limit lower=-0.785398 upper=0.610865 effort=100 velocity=1.0 -> lower=-0.785398 upper=0.610865 effort=100 velocity=2.0
- joint jLeftAnkle_roty: limit lower=-0.523599 upper=0.872665 effort=100 velocity=1.0 -> lower=-0.523599 upper=0.872665 effort=100 velocity=2.0
- joint jLeftAnkle_rotz: limit lower=-0.872665 upper=0.436332 effort=100 velocity=1.0 -> lower=-0.872665 upper=0.436332 effort=100 velocity=2.0
- joint jLeftBallFoot_roty: limit lower=-0.174533 upper=1.5708 effort=100 velocity=1.0 -> lower=-0.174533 upper=1.5708 effort=100 velocity=2.0
- joint jLeftC7Shoulder_rotx: limit lower=-0.6872665 upper=0.785398 effort=100 velocity=1.0 -> lower=-0.6872665 upper=0.785398 effort=100 velocity=2.0
- joint jLeftElbow_roty: limit lower=-1.5708 upper=1.48353 effort=100 velocity=1.0 -> (none); type revolute -> continuous
- joint jLeftElbow_rotz: limit lower=-2.53073 upper=0 effort=100 velocity=1.0 -> lower=-2.53073 upper=0 effort=100 velocity=2.0
- joint jLeftHip_rotx: limit lower=-0.523599 upper=0.785398 effort=100 velocity=1.0 -> lower=-0.523599 upper=0.785398 effort=100 velocity=2.0
- joint jLeftHip_roty: limit lower=-2.0944 upper=0.261799 effort=100 velocity=1.0 -> lower=-2.0944 upper=0.261799 effort=100 velocity=2.0
- joint jLeftHip_rotz: limit lower=-0.785398 upper=0.785398 effort=100 velocity=1.0 -> lower=-0.785398 upper=0.785398 effort=100 velocity=2.0
- joint jLeftKnee_roty: limit lower=0 upper=2.35619 effort=100 velocity=1.0 -> lower=0 upper=2.35619 effort=100 velocity=2.0
- joint jLeftKnee_rotz: limit lower=-0.523599 upper=0.698132 effort=100 velocity=1.0 -> lower=-0.523599 upper=0.698132 effort=100 velocity=2.0
- joint jLeftShoulder_rotx: limit lower=-1.5708 upper=2.35619 effort=100 velocity=1.0 -> lower=-1.5708 upper=2.35619 effort=100 velocity=2.0
- joint jLeftShoulder_roty: limit lower=-1.5708 upper=1.5708 effort=100 velocity=1.0 -> (none); type revolute -> continuous
- joint jLeftShoulder_rotz: limit lower=-3.14159 upper=0.785398 effort=100 velocity=1.0 -> lower=-3.14159 upper=0.785398 effort=100 velocity=2.0
- joint jLeftWrist_rotx: limit lower=-1.0472 upper=0.872665 effort=100 velocity=1.0 -> (none); type revolute -> continuous
- joint jLeftWrist_rotz: limit lower=-0.349066 upper=0.523599 effort=100 velocity=1.0 -> lower=-0.349066 upper=0.523599 effort=100 velocity=2.0
- joint jRightAnkle_rotx: limit lower=-0.610865 upper=0.785398 effort=100 velocity=1.0 -> lower=-0.610865 upper=0.785398 effort=100 velocity=2.0
- joint jRightAnkle_roty: limit lower=-0.523599 upper=0.872665 effort=100 velocity=1.0 -> lower=-0.523599 upper=0.872665 effort=100 velocity=2.0
- joint jRightAnkle_rotz: limit lower=-0.436332 upper=0.872665 effort=100 velocity=1.0 -> lower=-0.436332 upper=0.872665 effort=100 velocity=2.0
- joint jRightBallFoot_roty: limit lower=-0.174533 upper=1.5708 effort=100 velocity=1.0 -> lower=-0.174533 upper=1.5708 effort=100 velocity=2.0
- joint jRightC7Shoulder_rotx: limit lower=-0.785398 upper=0.0872665 effort=100 velocity=1.0 -> lower=-0.785398 upper=0.0872665 effort=100 velocity=2.0
- joint jRightElbow_roty: limit lower=-1.5708 upper=1.48353 effort=100 velocity=1.0 -> lower=-1.5708 upper=1.48353 effort=100 velocity=2.0
- joint jRightElbow_rotz: limit lower=0 upper=2.53073 effort=100 velocity=1.0 -> lower=0 upper=2.53073 effort=100 velocity=2.0
- joint jRightHip_rotx: limit lower=-0.785398 upper=0.523599 effort=100 velocity=1.0 -> lower=-0.785398 upper=0.523599 effort=100 velocity=2.0
- joint jRightHip_roty: limit lower=-2.0944 upper=0.261799 effort=100 velocity=1.0 -> lower=-2.0944 upper=0.261799 effort=100 velocity=2.0
- joint jRightHip_rotz: limit lower=-0.785398 upper=0.785398 effort=100 velocity=1.0 -> lower=-0.785398 upper=0.785398 effort=100 velocity=2.0
- joint jRightKnee_roty: limit lower=0 upper=2.35619 effort=100 velocity=1.0 -> lower=0 upper=2.35619 effort=100 velocity=2.0
- joint jRightKnee_rotz: limit lower=-0.698132 upper=0.523599 effort=100 velocity=1.0 -> lower=-0.698132 upper=0.523599 effort=100 velocity=2.0
- joint jRightShoulder_rotx: limit lower=-2.35619 upper=1.5708 effort=100 velocity=1.0 -> lower=-2.35619 upper=1.5708 effort=100 velocity=2.0
- joint jRightShoulder_roty: limit lower=-1.5708 upper=1.5708 effort=100 velocity=1.0 -> lower=-1.5708 upper=1.5708 effort=100 velocity=2.0
- joint jRightShoulder_rotz: limit lower=-0.785398 upper=3.14159 effort=100 velocity=1.0 -> lower=-0.785398 upper=3.14159 effort=100 velocity=2.0
- joint jRightWrist_rotx: limit lower=-0.872665 upper=1.0472 effort=100 velocity=1.0 -> lower=-0.872665 upper=1.0472 effort=100 velocity=2.0
- joint jRightWrist_rotz: limit lower=-0.523599 upper=0.349066 effort=100 velocity=1.0 -> lower=-0.523599 upper=0.349066 effort=100 velocity=2.0
- joint jT1C7_rotx: limit lower=-0.610865 upper=0.610865 effort=100 velocity=1.0 -> lower=-0.610865 upper=0.610865 effort=100 velocity=2.0
- joint jT1C7_roty: limit lower=-0.959931 upper=1.5708 effort=100 velocity=1.0 -> lower=-0.959931 upper=1.5708 effort=100 velocity=2.0
- joint jT1C7_rotz: limit lower=-1.22173 upper=1.22173 effort=100 velocity=1.0 -> lower=-1.22173 upper=1.22173 effort=100 velocity=2.0
- joint jT9T8_rotx: limit lower=-0.349066 upper=0.349066 effort=100 velocity=1.0 -> lower=-0.349066 upper=0.349066 effort=100 velocity=2.0
- joint jT9T8_roty: limit lower=-0.261799 upper=0.698132 effort=100 velocity=1.0 -> lower=-0.261799 upper=0.698132 effort=100 velocity=2.0
- joint jT9T8_rotz: limit lower=-0.610865 upper=0.610865 effort=100 velocity=1.0 -> lower=-0.610865 upper=0.610865 effort=100 velocity=2.0
